File: footprint try/new/new.kicad_pcb (KiCad board)
At the start: 2 copper layers, 55 parts

Commit message: add files
Parts:
- added S1: Keyswitch, Dome:7mm dome switch, F.Cu at (25.0, 23.5)
- added S10: Keyswitch, Dome:7mm dome switch, F.Cu at (198.2, 45.6)
- added S11: Keyswitch, Dome:7mm dome switch, F.Cu at (198.2, 63.7)
- added S12: Keyswitch, Dome:7mm dome switch, F.Cu at (198.2, 81.8)
- added S13: Keyswitch, Dome:7mm dome switch, F.Cu at (198.2, 99.9)
- added S14: Keyswitch, Dome:7mm dome switch, F.Cu at (198.2, 118.0)
- added S15: Keyswitch, Dome:7mm dome switch, F.Cu at (198.2, 136.1)
- added S16: Keyswitch, Dome:7mm dome switch, F.Cu at (198.2, 154.2)
- added S17: Keyswitch, Dome:7mm dome switch, F.Cu at (217.3, 27.5)
- added S18: Keyswitch, Dome:7mm dome switch, F.Cu at (217.3, 45.6)
- added S19: Keyswitch, Dome:7mm dome switch, F.Cu at (217.3, 63.7)
- added S2: Keyswitch, Dome:7mm dome switch, F.Cu at (49.5, 23.5)
- added S20: Keyswitch, Dome:7mm dome switch, F.Cu at (217.3, 81.8)
- added S21: Keyswitch, Dome:7mm dome switch, F.Cu at (217.3, 99.9)
- added S22: Keyswitch, Dome:7mm dome switch, F.Cu at (217.3, 118.0)
- added S23: Keyswitch, Dome:7mm dome switch, F.Cu at (217.3, 136.1)
- added S24: Keyswitch, Dome:7mm dome switch, F.Cu at (217.3, 154.2)
- added S25: Keyswitch, Dome:7mm dome switch, F.Cu at (236.4, 27.5)
- added S26: Keyswitch, Dome:7mm dome switch, F.Cu at (236.4, 45.6)
- added S27: Keyswitch, Dome:7mm dome switch, F.Cu at (236.4, 63.7)
- added S28: Keyswitch, Dome:7mm dome switch, F.Cu at (236.4, 81.8)
- added S29: Keyswitch, Dome:7mm dome switch, F.Cu at (236.4, 99.9)
- added S3: Keyswitch, Dome:7mm dome switch, F.Cu at (71.0, 23.5)
- added S30: Keyswitch, Dome:7mm dome switch, F.Cu at (236.4, 118.0)
- added S31: Keyswitch, Dome:7mm dome switch, F.Cu at (236.4, 136.1)
- added S32: Keyswitch, Dome:7mm dome switch, F.Cu at (236.4, 154.2)
- added S33: Keyswitch, Dome:7mm dome switch, F.Cu at (255.6, 27.5)
- added S34: Keyswitch, Dome:7mm dome switch, F.Cu at (255.6, 45.6)
- added S35: Keyswitch, Dome:7mm dome switch, F.Cu at (255.6, 63.7)
- added S36: Keyswitch, Dome:7mm dome switch, F.Cu at (255.6, 81.8)
- added S37: Keyswitch, Dome:7mm dome switch, F.Cu at (255.6, 99.9)
- added S38: Keyswitch, Dome:7mm dome switch, F.Cu at (255.6, 118.0)
- added S39: Keyswitch, Dome:7mm dome switch, F.Cu at (255.6, 136.1)
- added S4: Keyswitch, Dome:7mm dome switch, F.Cu at (179.0, 81.8)
- added S40: Keyswitch, Dome:7mm dome switch, F.Cu at (255.6, 154.2)
- added S41: Keyswitch, Dome:7mm dome switch, F.Cu at (274.8, 27.5)
- added S42: Keyswitch, Dome:7mm dome switch, F.Cu at (274.8, 45.6)
- added S43: Keyswitch, Dome:7mm dome switch, F.Cu at (274.8, 63.7)
- added S44: Keyswitch, Dome:7mm dome switch, F.Cu at (274.8, 81.8)
- added S45: Keyswitch, Dome:7mm dome switch, F.Cu at (274.8, 99.9)
- added S46: Keyswitch, Dome:7mm dome switch, F.Cu at (274.8, 118.0)
- added S47: Keyswitch, Dome:7mm dome switch, F.Cu at (274.8, 136.1)
- added S48: Keyswitch, Dome:7mm dome switch, F.Cu at (274.8, 154.2)
- added S49: Keyswitch, Dome:7mm dome switch, F.Cu at (293.9, 27.5)
- added S5: Keyswitch, Dome:7mm dome switch, F.Cu at (179.0, 99.9)
- added S50: Keyswitch, Dome:7mm dome switch, F.Cu at (293.9, 45.6)
- added S51: Keyswitch, Dome:7mm dome switch, F.Cu at (293.9, 63.7)
- added S52: Keyswitch, Dome:7mm dome switch, F.Cu at (293.9, 81.8)
- added S53: Keyswitch, Dome:7mm dome switch, F.Cu at (293.9, 99.9)
- added S54: Keyswitch, Dome:7mm dome switch, F.Cu at (293.9, 118.0)
- added S55: Keyswitch, Dome:7mm dome switch, F.Cu at (293.9, 136.1)
- added S6: Keyswitch, Dome:7mm dome switch, F.Cu at (179.0, 118.0)
- added S7: Keyswitch, Dome:7mm dome switch, F.Cu at (179.0, 136.1)
- added S8: Keyswitch, Dome:7mm dome switch, F.Cu at (179.0, 154.2)
- added S9: Keyswitch, Dome:7mm dome switch, F.Cu at (198.2, 27.5)
- moved D12 227.7 mm to (337.9, 63.1)
- moved D13 227.7 mm to (337.9, 66.5)
- moved D14 227.7 mm to (337.9, 69.8)
- moved D15 227.7 mm to (337.9, 73.2)
- moved D16 227.7 mm to (337.9, 76.5)
- moved D17 227.7 mm to (337.9, 79.8)
- moved D18 227.7 mm to (337.9, 83.2)
- moved D19 227.7 mm to (337.9, 86.5)
- moved D20 227.7 mm to (337.9, 89.9)
- moved D21 227.7 mm to (337.9, 93.2)
- moved D22 227.7 mm to (337.9, 96.6)
- moved D45 227.7 mm to (355.2, 63.1)
- moved D46 227.7 mm to (355.2, 66.5)
- moved D47 227.7 mm to (355.2, 69.8)
- moved D48 227.7 mm to (355.2, 73.2)
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