File: final_layout/final_layout.kicad_pcb (KiCad board)
At the start: 2 copper layers, 110 parts

Commit message: add layout for keyboard
Parts:
- removed D55: Diode, Diode_SMD:D_SOD-123
- removed S55: Keyswitch, Dome_05_30:Untitled_2
- added TP1: TestPoint, TestPoint:TestPoint_Pad_D1.5mm, B.Cu at (32.0, 144.0)
- added TP10: TestPoint, TestPoint:TestPoint_Pad_D1.5mm, B.Cu at (201.0, 86.0)
- added TP11: TestPoint, TestPoint:TestPoint_Pad_D1.5mm, B.Cu at (191.0, 104.0)
- added TP12: TestPoint, TestPoint:TestPoint_Pad_D1.5mm, B.Cu at (201.0, 122.0)
- added TP13: TestPoint, TestPoint:TestPoint_Pad_D1.5mm, B.Cu at (191.0, 139.0)
- added TP14: TestPoint, TestPoint:TestPoint_Pad_D1.5mm, B.Cu at (146.0, 144.0)
- added TP15: TestPoint, TestPoint:TestPoint_Pad_D1.5mm, B.Cu at (165.0, 144.0)
- added TP16: TestPoint, TestPoint:TestPoint_Pad_D1.5mm, B.Cu at (184.0, 144.0)
- added TP17: TestPoint, TestPoint:TestPoint_Pad_D1.5mm, B.Cu at (194.0, 127.0)
- added TP2: TestPoint, TestPoint:TestPoint_Pad_D1.5mm, B.Cu at (51.0, 144.0)
- added TP3: TestPoint, TestPoint:TestPoint_Pad_D1.5mm, B.Cu at (70.0, 144.0)
- added TP4: TestPoint, TestPoint:TestPoint_Pad_D1.5mm, B.Cu at (95.0, 147.0)
- added TP5: TestPoint, TestPoint:TestPoint_Pad_D1.5mm, B.Cu at (108.0, 130.0)
- added TP6: TestPoint, TestPoint:TestPoint_Pad_D1.5mm, B.Cu at (122.0, 147.0)
- added TP7: TestPoint, TestPoint:TestPoint_Pad_D1.5mm, B.Cu at (140.0, 28.0)
- added TP8: TestPoint, TestPoint:TestPoint_Pad_D1.5mm, B.Cu at (150.0, 46.0)
- added TP9: TestPoint, TestPoint:TestPoint_Pad_D1.5mm, B.Cu at (140.0, 64.0)
- added U1: Ag9905LP, joystick:joystick hole, F.Cu at (177.0, 42.0)
- D1, D10, D11, D12, D13, D14, D15, D16, D17, D18, D19, D2, D20, D21, D22, D23, D24, D25, D26, D27, D28, D29, D3, D30, D31, D32, D33, D34, D35, D36, D37, D38, D39, D4, D40, D41, D42, D43, D44, D45, D46, D47, D48, D49, D5, D50, D51, D52, D53, D54, D6, D7, D8, D9: footprint Diode_SMD:D_SOD-123 -> Diode_SMD:D_PowerDI-123; moved to B.Cu
- S1, S10, S11, S12, S13, S14, S15, S16, S17, S18, S19, S2, S20, S21, S22, S23, S24, S25, S26, S27, S28, S29, S3, S30, S31, S32, S33, S34, S35, S36, S37, S38, S39, S4, S40, S41, S42, S43, S44, S45, S46, S47, S48, S49, S5, S50, S51, S52, S53, S54, S6, S7, S8, S9: footprint Dome_05_30:Untitled_2 -> Dome_switch:7mm metal dome switch
- moved D47 435.2 mm to (32.0, 138.2), turned to 90 degrees
- moved D37 433.7 mm to (23.0, 121.2), turned to 90 degrees
- moved D48 416.0 mm to (51.0, 138.2), turned to 90 degrees
- moved D18 415.2 mm to (23.0, 85.2), turned to 90 degrees
- moved D28 414.7 mm to (32.0, 103.2), turned to 90 degrees
- moved D38 414.4 mm to (42.0, 121.2), turned to 90 degrees
- moved D49 396.8 mm to (70.0, 138.2), turned to 90 degrees
- moved D19 395.9 mm to (42.0, 85.2), turned to 90 degrees
- moved D29 395.4 mm to (51.0, 103.2), turned to 90 degrees
- moved D7 395.2 mm to (35.0, 45.1), turned to 90 degrees
- moved D39 395.1 mm to (61.0, 121.2), turned to 90 degrees
- moved D13 389.4 mm to (48.0, 59.1), turned to 90 degrees
- moved D20 376.7 mm to (61.0, 85.2), turned to 90 degrees
- moved D30 376.1 mm to (70.0, 103.2), turned to 90 degrees
- moved D40 375.9 mm to (80.0, 121.2), turned to 90 degrees
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Connections:
- D1 pad 1: row0 -> Net-(D1-K)
- D10 pad 1: row4 -> Net-(D10-K)
- D11 pad 1: row5 -> Net-(D10-K)
- D12 pad 1: row0 -> Net-(D10-K)
- D13 pad 1: row2 -> Net-(D13-K)
- D14 pad 1: row3 -> Net-(D13-K)
- D15 pad 1: row4 -> Net-(D13-K)
- D16 pad 1: row5 -> Net-(D13-K)
- D17 pad 1: row0 -> Net-(D13-K)
- D18 pad 1: row1 -> Net-(D18-K)
- D19 pad 1: row2 -> Net-(D18-K)
- D2 pad 1: row1 -> Net-(D1-K)
- D20 pad 1: row3 -> Net-(D18-K)
- D21 pad 1: row4 -> Net-(D18-K)
- D22 pad 1: row5 -> Net-(D18-K)
- D23 pad 1: row0 -> Net-(D18-K)
- D24 pad 1: row1 -> Net-(D18-K)
- D25 pad 1: row2 -> Net-(D18-K)
- D26 pad 1: row3 -> Net-(D18-K)
- D27 pad 1: row4 -> Net-(D18-K)
- D28 pad 1: row5 -> Net-(D28-K)
- D29 pad 1: row0 -> Net-(D28-K)
- D3 pad 1: row2 -> Net-(D1-K)
- D30 pad 1: row1 -> Net-(D28-K)
- D31 pad 1: row2 -> Net-(D28-K)
- D32 pad 1: row3 -> Net-(D28-K)
- D33 pad 1: row4 -> Net-(D28-K)
- D34 pad 1: row0 -> Net-(D28-K)
- D35 pad 1: row1 -> Net-(D28-K)
- D36 pad 1: row2 -> Net-(D28-K)
- D37 pad 1: row3 -> Net-(D37-K)
- D38 pad 1: row4 -> Net-(D37-K)
- D39 pad 1: row5 -> Net-(D37-K)
- D4 pad 1: row4 -> Net-(D1-K)
- D40 pad 1: row0 -> Net-(D37-K)
- D41 pad 1: row1 -> Net-(D37-K)
- D42 pad 1: row2 -> Net-(D37-K)
- D43 pad 1: row3 -> Net-(D37-K)
- D44 pad 1: row4 -> Net-(D37-K)
- D45 pad 1: row5 -> Net-(D37-K)
- D46 pad 1: row0 -> Net-(D37-K)
- D47 pad 1: row1 -> Net-(D47-K)
- D48 pad 1: row2 -> Net-(D47-K)
- D49 pad 1: row3 -> Net-(D47-K)
- D5 pad 1: row5 -> Net-(D1-K)
- D50 pad 1: row4 -> Net-(D47-K)
- D51 pad 1: row5 -> Net-(D47-K)
- D52 pad 1: row0 -> Net-(D47-K)
- D53 pad 1: row2 -> Net-(D47-K)
- D54 pad 1: row3 -> Net-(D47-K)
- D6 pad 1: row0 -> Net-(D1-K)
- D7 pad 1: row1 -> Net-(D10-K)
- D8 pad 1: row2 -> Net-(D10-K)
- D9 pad 1: row3 -> Net-(D10-K)
- S1 pad 1: Net-(D1-A) -> Net-(S1-Pad1)
- S1 pad 2: column0 -> Net-(D1-A)
- S10 pad 1: Net-(D10-A) -> Net-(S10-Pad1)
- S10 pad 2: column1 -> Net-(D10-A)
- S11 pad 1: Net-(D11-A) -> Net-(S11-Pad1)
- S11 pad 2: column1 -> Net-(D11-A)
- S12 pad 1: Net-(D12-A) -> Net-(S12-Pad1)
- S12 pad 2: column2 -> Net-(D12-A)
- S13 pad 1: Net-(D13-A) -> Net-(S1-Pad1)
- S13 pad 2: column2 -> Net-(D13-A)
- S14 pad 1: Net-(D14-A) -> Net-(S14-Pad1)
- S14 pad 2: column2 -> Net-(D14-A)
- S15 pad 1: Net-(D15-A) -> Net-(S10-Pad1)
- S15 pad 2: column2 -> Net-(D15-A)
- S16 pad 1: Net-(D16-A) -> Net-(S11-Pad1)
- S16 pad 2: column2 -> Net-(D16-A)
- S17 pad 1: Net-(D17-A) -> Net-(S12-Pad1)
- S17 pad 2: column3 -> Net-(D17-A)
- S18 pad 1: Net-(D18-A) -> Net-(S1-Pad1)
- S18 pad 2: column3 -> Net-(D18-A)
- S19 pad 1: Net-(D19-A) -> Net-(S19-Pad1)
- S19 pad 2: column3 -> Net-(D19-A)
- S2 pad 1: Net-(D2-A) -> Net-(S19-Pad1)
- S2 pad 2: column0 -> Net-(D2-A)
- S20 pad 1: Net-(D20-A) -> Net-(S14-Pad1)
- S20 pad 2: column3 -> Net-(D20-A)
- S21 pad 1: Net-(D21-A) -> Net-(S10-Pad1)
- S21 pad 2: column3 -> Net-(D21-A)
- S22 pad 1: Net-(D22-A) -> Net-(S11-Pad1)
- S22 pad 2: column3 -> Net-(D22-A)
- S23 pad 1: Net-(D23-A) -> Net-(S12-Pad1)
- S23 pad 2: column4 -> Net-(D23-A)
- S24 pad 1: Net-(D24-A) -> Net-(S24-Pad1)
- S24 pad 2: column4 -> Net-(D24-A)
- S25 pad 1: Net-(D25-A) -> Net-(S25-Pad1)
- S25 pad 2: column4 -> Net-(D25-A)
- S26 pad 1: Net-(D26-A) -> Net-(S26-Pad1)
- S26 pad 2: column4 -> Net-(D26-A)
- S27 pad 1: Net-(D27-A) -> Net-(S27-Pad1)
- S27 pad 2: column4 -> Net-(D27-A)
- S28 pad 1: Net-(D28-A) -> Net-(S1-Pad1)
- S28 pad 2: column4 -> Net-(D28-A)
- S29 pad 1: Net-(D29-A) -> Net-(S19-Pad1)
- S29 pad 2: column5 -> Net-(D29-A)
- S3 pad 1: Net-(D3-A) -> Net-(S14-Pad1)
- S3 pad 2: column0 -> Net-(D3-A)
- S30 pad 1: Net-(D30-A) -> Net-(S14-Pad1)
- S30 pad 2: column5 -> Net-(D30-A)
- S31 pad 1: Net-(D31-A) -> Net-(S10-Pad1)
- S31 pad 2: column5 -> Net-(D31-A)
- S32 pad 1: Net-(D32-A) -> Net-(S11-Pad1)
- S32 pad 2: column5 -> Net-(D32-A)
- S33 pad 1: Net-(D33-A) -> Net-(S12-Pad1)
- S33 pad 2: column5 -> Net-(D33-A)
- S34 pad 1: Net-(D34-A) -> Net-(S24-Pad1)
- S34 pad 2: column6 -> Net-(D34-A)
- S35 pad 1: Net-(D35-A) -> Net-(S25-Pad1)
- S35 pad 2: column6 -> Net-(D35-A)
- S36 pad 1: Net-(D36-A) -> Net-(S26-Pad1)
- S36 pad 2: column6 -> Net-(D36-A)
- S37 pad 1: Net-(D37-A) -> Net-(S1-Pad1)
- S37 pad 2: column6 -> Net-(D37-A)
- S38 pad 1: Net-(D38-A) -> Net-(S19-Pad1)
- S38 pad 2: column6 -> Net-(D38-A)
- S39 pad 1: Net-(D39-A) -> Net-(S14-Pad1)
- S39 pad 2: column6 -> Net-(D39-A)
- S4 pad 1: Net-(D4-A) -> Net-(S10-Pad1)
- S4 pad 2: column0 -> Net-(D4-A)
- S40 pad 1: Net-(D40-A) -> Net-(S10-Pad1)
- S40 pad 2: column7 -> Net-(D40-A)
- S41 pad 1: Net-(D41-A) -> Net-(S11-Pad1)
- S41 pad 2: column7 -> Net-(D41-A)
- S42 pad 1: Net-(D42-A) -> Net-(S12-Pad1)
- S42 pad 2: column7 -> Net-(D42-A)
- S43 pad 1: Net-(D43-A) -> Net-(S24-Pad1)
- S43 pad 2: column7 -> Net-(D43-A)
- S44 pad 1: Net-(D44-A) -> Net-(S25-Pad1)
- S44 pad 2: column7 -> Net-(D44-A)
- S45 pad 1: Net-(D45-A) -> Net-(S26-Pad1)
- S45 pad 2: column7 -> Net-(D45-A)
- S46 pad 1: Net-(D46-A) -> Net-(S27-Pad1)
- S46 pad 2: column8 -> Net-(D46-A)
- S47 pad 1: Net-(D47-A) -> Net-(S1-Pad1)
- S47 pad 2: column8 -> Net-(D47-A)
- S48 pad 1: Net-(D48-A) -> Net-(S19-Pad1)
- S48 pad 2: column8 -> Net-(D48-A)
- S49 pad 1: Net-(D49-A) -> Net-(S14-Pad1)
- S49 pad 2: column8 -> Net-(D49-A)
- S5 pad 1: Net-(D5-A) -> Net-(S11-Pad1)
- S5 pad 2: column0 -> Net-(D5-A)
- S50 pad 1: Net-(D50-A) -> Net-(S10-Pad1)
- S50 pad 2: column8 -> Net-(D50-A)
- S51 pad 1: Net-(D51-A) -> Net-(S12-Pad1)
- S51 pad 2: column8 -> Net-(D51-A)
- S52 pad 1: Net-(D52-A) -> Net-(S24-Pad1)
- S52 pad 2: column9 -> Net-(D52-A)
- S53 pad 1: Net-(D53-A) -> Net-(S25-Pad1)
- S53 pad 2: column9 -> Net-(D53-A)
- S54 pad 1: Net-(D54-A) -> Net-(S26-Pad1)
- S54 pad 2: column9 -> Net-(D54-A)
- S6 pad 1: Net-(D6-A) -> Net-(S12-Pad1)
- S6 pad 2: column1 -> Net-(D6-A)
- S7 pad 1: Net-(D7-A) -> Net-(S1-Pad1)
- S7 pad 2: column1 -> Net-(D7-A)
- S8 pad 1: Net-(D8-A) -> Net-(S19-Pad1)
- S8 pad 2: column1 -> Net-(D8-A)
- S9 pad 1: Net-(D9-A) -> Net-(S14-Pad1)
- S9 pad 2: column1 -> Net-(D9-A)
