File: second_pcb/_autosave-second_pcb.kicad_pcb (KiCad board)
At the start: 2 copper layers, 99.2 x 69.6 mm, 194 parts, among them SW1 SW_Nidec_CAS-120A1, U1 MIC29502WU, U10 CJ432, U11 CJ432, U12 CJ432, U13 CJ432, U14 CJ432, U15 CJ432, U16 CJ432, U17 CJ432, U18 CJ432, U19 CJ432, U2 CJ432, U20 CJ432, U21 CJ432, U22 CJ432, U23 CJ432, U24 CJ432, U25 CJ432, U26 CJ432, U27 CJ432, U28 CJ432, U29 CJ432, U3 CJ432, U30 CJ432, U31 CJ432, U32 CJ432, U33 CJ432, U34 CJ432, U35 CJ432, U36 CJ432, U37 CJ432, U38 CJ432, U39 CJ432, U4 CJ432, U40 CJ432, U41 CJ432, U42 CJ432, U43 CJ432, U44 CJ432, U45 CJ432, U46 CJ432, U47 CJ432, U48 CJ432, U49 CJ432, U5 CJ432, U50 CJ432, U51 CJ432, U52 CJ432, U53 CJ432, U54 CJ432, U55 CJ432, U56 CJ432, U57 CJ432, U58 CJ432, U59 CJ432, U6 CJ432, U60 CJ432, U61 CJ432, U7 CJ432, U8 CJ432, U9 CJ432

Commit message: add a lot of things
Parts:
- moved D1 87.2 mm to (29.9, 121.1)
- moved D13 87.2 mm to (41.2, 134.4)
- moved D14 87.2 mm to (54.1, 135.5)
- moved D15 87.2 mm to (62.7, 135.5)
- moved D16 87.2 mm to (71.4, 135.5)
- moved D17 87.2 mm to (80.0, 135.5)
- moved D2 87.2 mm to (41.1, 125.1)
- moved D26 87.2 mm to (99.5, 144.2)
- moved D27 87.2 mm to (108.1, 144.2)
- moved D35 87.2 mm to (95.0, 151.1)
- moved D47 87.2 mm to (34.5, 165.0)
- moved D48 87.2 mm to (43.1, 165.0)
- moved D49 87.2 mm to (51.8, 165.0)
- moved D52 87.2 mm to (86.3, 165.0)
- moved D53 87.2 mm to (95.0, 165.0)
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Routing:
- net Net-(S27-Pad1): track 18.2 -> 15.3 mm
Other:
- board outline removed
