File: second_pcb/second_pcb.kicad_sch (KiCad schematic)
At the start: 195 parts, among them SW1 SW_Nidec_CAS-120A1, U1 MIC29502WU, U10 CJ432, U11 CJ432, U12 CJ432, U13 CJ432, U14 CJ432, U15 CJ432, U16 CJ432, U17 CJ432, U18 CJ432, U19 CJ432, U2 CJ432, U20 CJ432, U21 CJ432, U22 CJ432, U23 CJ432, U24 CJ432, U25 CJ432, U26 CJ432, U27 CJ432, U28 CJ432, U29 CJ432, U3 CJ432, U30 CJ432, U31 CJ432, U32 CJ432, U33 CJ432, U34 CJ432, U35 CJ432, U36 CJ432, U37 CJ432, U38 CJ432, U39 CJ432, U4 CJ432, U40 CJ432, U41 CJ432, U42 CJ432, U43 CJ432, U44 CJ432, U45 CJ432, U46 CJ432, U47 CJ432, U48 CJ432, U49 CJ432, U5 CJ432, U50 CJ432, U51 CJ432, U52 CJ432, U53 CJ432, U54 CJ432, U55 CJ432, U56 CJ432, U57 CJ432, U58 CJ432, U59 CJ432, U6 CJ432, U60 CJ432, U61 CJ432, U62 CJ432, U7 CJ432, U8 CJ432, U9 CJ432

Commit message: full size keyboard
Parts:
- U62: footprint lettersAndNumbers:Esc -> custom_footprints:LCD
Connections:
- net at D7.2 (A): now also S7.1; no longer S7.2
- net at S19.1, S29.1, S38.1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: now also S2.2, S8.2; no longer S2.1, S8.1
- net at D2.2 (A): now also S2.1; no longer S2.2
- net at S1.1, S18.1, S28.1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: now also S13.2, S7.2; no longer S13.1, S7.1
- net at D13.2 (A): now also S13.1; no longer S13.2
- net at D8.2 (A): now also S8.1; no longer S8.2
Other:
- moved on the sheet: S13, S2, S7, S8
Changed lines of the file:
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@@
 	)
 	(junction
-		(at 26.67 54.61)
-		(diameter 0)
-		(color 0 0 0 0)
-	)
-	(junction
 		(at 81.28 115.57)
 		(diameter 0)
@@
 	)
 	(junction
+		(at 43.18 54.61)
+		(diameter 0)
+		(color 0 0 0 0)
+	)
+	(junction
 		(at 59.69 146.05)
 		(diameter 0)
@@
 	)
 	(junction
+		(at 26.67 78.74)
+		(diameter 0)
+		(color 0 0 0 0)
+	)
+	(junction
 		(at 81.28 67.31)
 		(diameter 0)
@@
 	)
 	(junction
-		(at 26.67 78.74)
-		(diameter 0)
-		(color 0 0 0 0)
-	)
-	(junction
 		(at 114.3 115.57)
 		(diameter 0)
@@
 	)
 	(junction
+		(at 26.67 54.61)
+		(diameter 0)
+		(color 0 0 0 0)
+	)
+	(junction
 		(at 59.69 78.74)
 		(diameter 0)
@@
 	)
 	(junction
+		(at 43.18 31.75)
+		(diameter 0)
+		(color 0 0 0 0)
+	)
+	(junction
 		(at 64.77 91.44)
 		(diameter 0)
@@
 	)
 	(junction
-		(at 43.18 31.75)
-		(diameter 0)
-		(color 0 0 0 0)
-	)
-	(junction
 		(at 147.32 102.87)
 		(diameter 0)
@@
 	)
 	(junction
-		(at 43.18 54.61)
-		(diameter 0)
-		(color 0 0 0 0)
-	)
-	(junction
 		(at 152.4 182.88)
 		(diameter 0)
@@
 	(wire
 		(pts
-			(xy 26.67 31.75) (xy 26.67 54.61)
+			(xy 109.22 31.75) (xy 109.22 54.61)
 		)
 		(stroke
@@
 	(wire
 		(pts
-			(xy 109.22 31.75) (xy 109.22 54.61)
+			(xy 76.2 31.75) (xy 76.2 54.61)
 		)
 		(stroke
@@
 	(wire
 		(pts
-			(xy 76.2 31.75) (xy 76.2 54.61)
+			(xy 187.96 49.53) (xy 204.47 49.53)
 		)
 		(stroke
@@
 	(wire
 		(pts
-			(xy 187.96 49.53) (xy 204.47 49.53)
+			(xy 168.91 158.75) (xy 185.42 158.75)
 		)
 		(stroke
@@
 	(wire
 		(pts
-			(xy 168.91 158.75) (xy 185.42 158.75)
+			(xy 114.3 158.75) (xy 135.89 158.75)
 		)
 		(stroke
@@
 	(wire
 		(pts
-			(xy 114.3 158.75) (xy 135.89 158.75)
+			(xy 26.67 54.61) (xy 26.67 78.74)
 		)
 		(stroke
@@
 	(wire
 		(pts
+			(xy 26.67 78.74) (xy 26.67 102.87)
+		)
+		(stroke
+			(width 0)
+			(type default)
+		)
+	)
+	(wire
+		(pts
 			(xy 96.52 44.45) (xy 114.3 44.45)
 		)
@@
 	(wire
 		(pts
-			(xy 26.67 54.61) (xy 26.67 78.74)
+			(xy 26.67 31.75) (xy 26.67 54.61)
 		)
 		(stroke
@@
 	(wire
 		(pts
-			(xy 81.28 67.31) (xy 96.52 67.31)
-		)
-		(stroke
-			(width 0)
-			(type default)
-		)
-	)
-	(wire
-		(pts
 			(xy 43.18 54.61) (xy 43.18 102.87)
 		)
@@
 	(wire
 		(pts
-			(xy 31.75 158.75) (xy 48.26 158.75)
+			(xy 81.28 67.31) (xy 96.52 67.31)
 		)
 		(stroke
@@
 	(wire
 		(pts
-			(xy 147.32 78.74) (xy 147.32 102.87)
+			(xy 43.18 31.75) (xy 43.18 54.61)
 		)
 		(stroke
@@
 	(wire
 		(pts
-			(xy 163.83 102.87) (xy 163.83 125.73)
+			(xy 31.75 158.75) (xy 48.26 158.75)
 		)
 		(stroke
@@
 	(wire
 		(pts
-			(xy 180.34 102.87) (xy 180.34 146.05)
+			(xy 147.32 78.74) (xy 147.32 102.87)
 		)
 		(stroke
@@
 	(wire
 		(pts
-			(xy 109.22 25.4) (xy 109.22 31.75)
+			(xy 163.83 102.87) (xy 163.83 125.73)
 		)
 		(stroke
@@
 	(wire
 		(pts
-			(xy 43.18 31.75) (xy 43.18 54.61)
+			(xy 180.34 102.87) (xy 180.34 146.05)
 		)
 		(stroke
@@
 	(wire
 		(pts
-			(xy 26.67 78.74) (xy 26.67 102.87)
+			(xy 109.22 25.4) (xy 109.22 31.75)
 		)
 		(stroke
@@
 	(symbol
 		(lib_id "ScottoKeebs:Placeholder_Keyswitch")
-		(at 29.21 57.15 0)
+		(at 29.21 57.15 180)
 		(unit 1)
 		(exclude_from_sim no)
@@
 	(symbol
 		(lib_id "ScottoKeebs:Placeholder_Keyswitch")
-		(at 29.21 81.28 0)
+		(at 29.21 81.28 180)
 		(unit 1)
 		(exclude_from_sim no)
@@
 	)
 	(symbol
+		(lib_id "Reference_Voltage:CJ432")
+		(at 252.73 153.67 0)
+		(unit 1)
+		(exclude_from_sim no)
+		(in_bom yes)
+		(on_board yes)
+		(dnp no)
+		(fields_autoplaced yes)
+		(property "Reference" "U62"
+			(at 252.73 157.48 0)
+			(effects
+				(font
+					(size 1.27 1.27)
+				)
+			)
+		)
+		(property "Value" "CJ432"
+			(at 252.73 160.02 0)
+			(effects
+				(font
+					(size 1.27 1.27)
+				)
+			)
+		)
+		(property "Footprint" "custom_footprints:LCD"
+			(at 252.73 157.48 0)
+			(effects
+				(font
+					(size 1.27 1.27)
+					(italic yes)
+				)
+				(hide yes)
+			)
+		)
+		(property "Datasheet" "http://www.cj-elec.com/txUpfile/20134181474991806.pdf"
+			(at 252.73 153.67 0)
+			(effects
+				(font
+					(size 1.27 1.27)
+					(italic yes)
+				)
+				(hide yes)
+			)
+		)
+		(property "Description" "Shunt Regulator, SOT-23"
+			(at 252.73 153.67 0)
+			(effects
+				(font
+					(size 1.27 1.27)
+				)
+				(hide yes)
+			)
+		)
+		(pin "1"
+		)
+		(pin "3"
+		)
+		(pin "2"
+		)
+		(instances
+			(project "second_pcb"
+				(path "/fba27e40-e473-4210-a509-ee0b8da09b69"
+					(reference "U62")
+					(unit 1)
+				)
+			)
+		)
+	)
+	(symbol
 		(lib_id "ScottoKeebs:Placeholder_Keyswitch")
 		(at 45.72 128.27 0)
@@
 	(symbol
 		(lib_id "ScottoKeebs:Placeholder_Keyswitch")
-		(at 45.72 57.15 0)
+		(at 45.72 57.15 180)
 		(unit 1)
 		(exclude_from_sim no)
@@
 	(symbol
 		(lib_id "Reference_Voltage:CJ432")
-		(at 252.73 140.97 0)
-		(unit 1)
-		(exclude_from_sim no)
-		(in_bom yes)
-		(on_board yes)
-		(dnp no)
-		(fields_autoplaced yes)
-		(property "Reference" "U62"
-			(at 252.73 144.78 0)
-			(effects
-				(font
-					(size 1.27 1.27)
-				)
-			)
-		)
-		(property "Value" "CJ432"
-			(at 252.73 147.32 0)
-			(effects
-				(font
-					(size 1.27 1.27)
-				)
-			)
-		)
-		(property "Footprint" "lettersAndNumbers:Esc"
-			(at 252.73 144.78 0)
-			(effects
-				(font
-					(size 1.27 1.27)
-					(italic yes)
-				)
-				(hide yes)
-			)
-		)
-		(property "Datasheet" "http://www.cj-elec.com/txUpfile/20134181474991806.pdf"
-			(at 252.73 140.97 0)
-			(effects
-				(font
-					(size 1.27 1.27)
-					(italic yes)
-				)
-				(hide yes)
-			)
-		)
-		(property "Description" "Shunt Regulator, SOT-23"
-			(at 252.73 140.97 0)
-			(effects
-				(font
-					(size 1.27 1.27)
-				)
-				(hide yes)
-			)
-		)
-		(pin "1"
-		)
-		(pin "3"
-		)
-		(pin "2"
-		)
-		(instances
-			(project "second_pcb"
-				(path "/fba27e40-e473-4210-a509-ee0b8da09b69"
-					(reference "U62")
-					(unit 1)
-				)
-			)
-		)
-	)
-	(symbol
-		(lib_id "Reference_Voltage:CJ432")
 		(at 265.43 106.68 0)
 		(unit 1)
@@
 	(symbol
 		(lib_id "ScottoKeebs:Placeholder_Keyswitch")
-		(at 45.72 34.29 0)
+		(at 45.72 34.29 180)
 		(unit 1)
 		(exclude_from_sim no)
