File: full size keyboard/_autosave-full size keyboard.kicad_pcb (KiCad board)
At the start: 2 copper layers, 112.2 x 143.1 mm, 110 parts, among them SW1 SW_Nidec_CAS-120A1, U1 MIC29502WU, U15 CJ432, U16 CJ432, U17 CJ432, U19 CJ432, U2 CJ432, U20 CJ432, U21 CJ432, U23 CJ432, U24 CJ432, U25 CJ432, U3 CJ432, U38 CJ432, U39 CJ432, U40 CJ432, U42 CJ432, U43 CJ432, U44 CJ432, U45 CJ432, U46 CJ432, U51 CJ432, U52 CJ432, U53 CJ432, U55 CJ432, U57 CJ432, U59 CJ432, U60 CJ432, U62 CJ432

Commit message: changes
Parts:
- added S1: Keyswitch, custom_footprints:8mm, F.Cu at (137.5, 119.3)
- moved S46 5.24 mm to (132.4, 171.6)
Routing:
- net Net-(S27-Pad1): track 1.56 -> 0.00 mm
